File: Penta_OctoWS2811.kicad_pcb (KiCad board)
At the start: 2 copper layers, 91.5 x 104.5 mm, 93 parts, among them J1 Screw_Terminal_01x03, J10 RJ45, J11 RJ45, J12 J1B1211CCD, J13 Header 2x3 2mm, J14 Conn_01x24, J15 Conn_01x24, J16 Conn_01x01, J2 RJ45, J3 RJ45, J4 RJ45, J5 RJ45, J6 RJ45, J7 RJ45, J8 RJ45, J9 RJ45, U1 74HCT245, U2 74HCT245, U3 NCP1117-5.0_SOT223, U4 Teensy4.1, U5 74HCT245, U6 74HCT245, U7 74HCT245

Commit message: Fix VUSB diode. Diode from VIN to +5V was unnecessary, now using 2 parallel diodes from VUSB to VIN and tied VIN to +5V. Also fixed board name silkscreen typo.
Parts:
- D1: value BAT54S -> BAT54C
- moved C8 1.20 mm to (146.0, 39.8)
- moved D1 1.17 mm to (149.0, 39.8), turned to 180 degrees
Connections:
- net V_LED renamed VLED
- C8 pad 2: /t48 -> +5V
- D1 pad 2: /t48 -> /t49
- J15 pad 1: /t48 -> +5V
- U4 pad 48: /t48 -> +5V
Routing:
- net +5V: track 265.2 -> 279.3 mm
- net /t48: track 12.2 -> 0.00 mm
- net GND: track 18.7 -> 24.0 mm, vias 151 -> 152
- net /t49: track 3.98 -> 6.18 mm
Other:
- board text added: "Teensy 4.0/4.1 Penta-OctoWS2811 Adapter"
- board text removed: "Teensy 4.0/4.1 Penta-OctoWC2811 Adapter"
