File: Penta_OctoWS2811.kicad_sch (KiCad schematic)
At the start: 92 parts, among them J1 Screw_Terminal_01x03, J10 RJ45, J11 RJ45, J12 J1B1211CCD, J13 Header 2x3 2mm, J14 Conn_01x24, J15 Conn_01x24, J16 Conn_01x01, J2 RJ45, J3 RJ45, J4 RJ45, J5 RJ45, J6 RJ45, J7 RJ45, J8 RJ45, J9 RJ45, U1 74HCT245, U2 74HCT245, U3 NCP1117-5.0_SOT223, U4 Teensy4.1, U5 74HCT245, U6 74HCT245, U7 74HCT245

Commit message: Fix VUSB diode. Diode from VIN to +5V was unnecessary, now using 2 parallel diodes from VUSB to VIN and tied VIN to +5V. Also fixed board name silkscreen typo.
Parts:
- removed D1: BAT54S, Package_TO_SOT_SMD:SOT-23, symbol Diode:BAT54S
- added D1: BAT54C, Package_TO_SOT_SMD:SOT-23, symbol Diode:BAT54C
Connections:
- net t48 is gone; now on net +5V: C8.2, J15.1 (Pin_1), U4.48 (VIN)
- net +5V: now also D1.3
- net t49: now also D1.1, D1.2
- net V_LED renamed VLED
Other:
- note added: "Cutting VUSB jumper and installing VUSB pin allows Teensy and board to be powered from USB -or- VLED"
- note added: "VLED up to 12V (e.g. for use with WS2815 LEDs) If using 5V LEDs (WS2812b), bridge JP3 to power Teensy directly from 5V supply"
- note removed: "Cutting VUSB jumper and installing VUSB pin allows Teensy and board to be powered from USB -or- V_LED"
- note removed: "V_LED up to 12V (e.g. for use with WS2815 LEDs) If using 5V LEDs (WS2812b), bridge JP3 to power Teensy directly from 5V supply"
- moved on the sheet: C8
